File: CAN-Bus-Interface.brd (EAGLE design)
At the start: 50.8 x 40.4 mm, 18 parts, among them J1 M13, J4 MST4V, U1 MCP2515-P, U2 MCP2551-P

Commit message: added values for connectors
Parts:
- J1: value M13 -> 0.100
- LED1: value (none) -> O
- LED2: value (none) -> G
- LED3: value (none) -> B

Commit message: added values for connectors
Parts:
- CANPWR: value (none) -> 0.100
Changed lines of the file:
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@@
 </element>
 <element name="J1" library="SparkFun" package="1X13" value="0.100" x="33.02" y="2.54" smashed="yes" rot="R180"/>
-<element name="CANPWR" library="pinhead" package="1X02" value="" x="2.794" y="27.432" smashed="yes" rot="R90">
+<element name="CANPWR" library="pinhead" package="1X02" value="0.100" x="2.794" y="27.432" smashed="yes" rot="R90">
 <attribute name="NAME" x="2.0828" y="23.9522" size="1.27" layer="25" ratio="10" rot="R270"/>
 <attribute name="VALUE" x="5.969" y="24.892" size="1.27" layer="27" rot="R90"/>

Commit message: added values for connectors
Parts:
- TERM: value (none) -> 0.100
Changed lines of the file:
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@@
 <attribute name="VALUE" x="44.958" y="14.7066" size="0.8128" layer="27" font="vector" ratio="10" rot="R180"/>
 </element>
-<element name="TERM" library="pinhead" package="1X02" value="" x="27.432" y="38.1" smashed="yes">
+<element name="TERM" library="pinhead" package="1X02" value="0.100" x="27.432" y="38.1" smashed="yes">
 <attribute name="NAME" x="31.6992" y="35.4838" size="1.27" layer="25" font="vector" ratio="10" rot="R90"/>
 <attribute name="VALUE" x="24.892" y="34.925" size="1.27" layer="27"/>

Commit message: normalized values
Parts:
- J4: value MST4V -> 0.200
Changed lines of the file:
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@@
 <attribute name="VALUE" x="24.892" y="34.925" size="1.27" layer="27"/>
 </element>
-<element name="J4" library="con-phoenix-508" package="MSTBV4" value="MST4V" x="11.176" y="36.068" smashed="yes"/>
+<element name="J4" library="con-phoenix-508" package="MSTBV4" value="0.200" x="11.176" y="36.068" smashed="yes"/>
 <element name="R1" library="rcl" package="0204/5" value="470R" x="34.798" y="28.956" smashed="yes">
 <attribute name="NAME" x="33.909" y="26.924" size="0.8128" layer="25" font="vector"/>
